File: hardware/rev-b/main/main-revb.kicad_pcb (KiCad board)
At the start: 4 copper layers, 53.4 x 92.4 mm, 142 parts, among them J1 PicoBlade2Pin, J2 FH34SRJ_4S_0P5SH_99, J3 53261-0371, J5 USB_C_Receptacle_2_0, SW1 SKTDLDE010, SW2 SKTDLDE010, SW3 TactileSwitchSPST, SW4 TactileSwitchSPST, SW5 SKTDLDE010, SW6 SKTDLDE010, U1 NS4150B, U10 TPS22918, U2 TPS22918, U20 USBLC6, U3 H0216F002AM, U4 W25Q128JV, U5 SF32LB525UC6, U6 BQ24073RGTR, U7 RT6150B, U8 RT6150B, Y1 Crystal_4pad

Commit message: Set Rev B charging to 0.5C and add the Chinese assembly BOM
Parts:
- R37: value 2.55kohm -> 3.6kohm
Changed lines of the file:
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@@
 			)
 		)
-		(property "Description" "TI bq24073 1-cell Li-ion linear charger with power path (DPPM), VQFN-16 3x3 RGT; USB500, ISET 2.55k, TD/CE/EN2 low, EN1=OUT, TMR open"
+		(property "Description" "TI bq24073 1-cell Li-ion linear charger with power path (DPPM), VQFN-16 3x3 RGT; USB500, ISET 3.6k (247 mA, 0.5 C of the 500 mAh cell), TD/CE/EN2 low, EN1=OUT, TMR open"
 			(at 0 0 0)
 			(layer "F.Fab")
@@
 			)
 		)
-		(property "Value" "2.55kohm"
+		(property "Value" "3.6kohm"
 			(at 0 0 90)
 			(layer "F.Fab")
@@
 		)
 		(embedded_fonts no)
-		(model "${KIPRJMOD}/../models/RC0402FR-072K55L.step"
+		(model "${KIPRJMOD}/../models/RC0402FR-073K6L.step"
 			(offset
 				(xyz 0 0 0)
